Commit message: ✨ feat:
for fisheye calib

File: urdf/robot.urdf.xacro (robot description, xacro)
@@ -6,5 +6,5 @@
 			<origin xyz="0 0 0" rpy="0 0 0"/>
 			<geometry>
-				<box size="1.0 1.0 1.0"/>
+				<box size="0.2 0.2 0.2"/>
 			</geometry>
 		</collision>
@@ -12,10 +12,10 @@
 			<origin xyz="0 0 0" rpy="0 0 0" />
 			<geometry>
-				<box size="1.0 1.0 1.0" />
+				<box size="0.2 0.2 0.2" />
 			</geometry>
 		</visual>
 		<inertial>
 			<mass value="1.0" />
-			<inertia ixx="0.0833333" ixy = "0" ixz = "0" iyy="0.0833333" iyz= "0" izz="0.0833333" />
+			<inertia ixx="0.0066667" ixy = "0" ixz = "0" iyy="0.0066667" iyz= "0" izz="0.0066667" />
 		</inertial>
 	</link>
@@ -35,5 +35,5 @@
 		</plugin>
 	</gazebo>
-    <link name="imu_link"/>
+    <!-- <link name="imu_link"/>
     <joint name="imu_joint" type="fixed">
         <origin xyz="0.0 0.0 0.0" rpy="0 0 0"/>
@@ -53,10 +53,10 @@
             <headingGaussianNoise>0.0</headingGaussianNoise>
         </plugin>
-    </gazebo>
+    </gazebo> -->
     <!-- velodyne and its parameters-->
-    <xacro:include filename="$(find obj_with_6dof)/urdf/velodyne.xacro"/>
+    <!-- <xacro:include filename="$(find obj_with_6dof)/urdf/velodyne.xacro"/>
 	<xacro:VLP name="rslidar16" topic="lidar_points" organize_cloud="true" hz="10" gpu="true" visualize="false">
 		<origin xyz="0.1 0.2 0.3" rpy="0 0 ${M_PI}" />
-	</xacro:VLP>
+	</xacro:VLP> -->
     <!-- <xacro:include filename="$(find obj_with_6dof)/urdf/velodyne.xacro"/>
 	<xacro:VLP name="rslidar16" topic="lidar_points" organize_cloud="true" hz="10" gpu="true" visualize="false">
@@ -68,3 +68,17 @@
 		<origin xyz="0.1 0.1 0.1" rpy="0 0 0" />
 	</xacro:Macro_CameraROS> -->
+    <xacro:include filename="$(find obj_with_6dof)/urdf/fisheye.xacro"/>
+	<xacro:macro_fisheye name="front_cam" parent="base_link" hfov="1.92" hz="10" width="800" height="768">
+		<origin xyz="0.2 0 0" rpy="0 0 0" />
+	</xacro:macro_fisheye>
+    <!-- left -->
+    <xacro:include filename="$(find obj_with_6dof)/urdf/fisheye.xacro"/>
+	<xacro:macro_fisheye name="left_cam" parent="base_link" hfov="1.92" hz="10" width="800" height="768">
+		<origin xyz="0 0.2 0" rpy="0 0 ${M_PI/2}" />
+	</xacro:macro_fisheye>
+    <!-- right -->
+    <!-- <xacro:include filename="$(find obj_with_6dof)/urdf/fisheye.xacro"/>
+	<xacro:macro_fisheye name="left_cam" parent="base_link" hfov="1.92" hz="10" width="800" height="768">
+		<origin xyz="0 -0.2 0" rpy="0 0 -${M_PI/2}" />
+	</xacro:macro_fisheye> -->
 </robot>

Commit message: ✨ feat:
finish all 4 fisheyes and output vis

File: urdf/robot.urdf.xacro (robot description, xacro)
@@ -78,7 +78,12 @@
 	</xacro:macro_fisheye>
     <!-- right -->
-    <!-- <xacro:include filename="$(find obj_with_6dof)/urdf/fisheye.xacro"/>
-	<xacro:macro_fisheye name="left_cam" parent="base_link" hfov="1.92" hz="10" width="800" height="768">
+    <xacro:include filename="$(find obj_with_6dof)/urdf/fisheye.xacro"/>
+	<xacro:macro_fisheye name="right_cam" parent="base_link" hfov="1.92" hz="10" width="800" height="768">
 		<origin xyz="0 -0.2 0" rpy="0 0 -${M_PI/2}" />
-	</xacro:macro_fisheye> -->
+	</xacro:macro_fisheye>
+    <!-- back -->
+    <xacro:include filename="$(find obj_with_6dof)/urdf/fisheye.xacro"/>
+	<xacro:macro_fisheye name="back_cam" parent="base_link" hfov="1.92" hz="10" width="800" height="768">
+		<origin xyz="-0.2 0 0" rpy="0 0 ${M_PI}" />
+	</xacro:macro_fisheye>
 </robot>

Commit message: ✨ feat: finish avia urdf

File: urdf/robot.urdf.xacro (robot description, xacro)
@@ -2,9 +2,18 @@
 <robot name="robot" xmlns:xacro="http://ros.org/wiki/xacro">
 	<xacro:property name="M_PI" value="3.14159265358979"/>
+    <xacro:property name="cam_size" value="0.1"/>
+    <xacro:macro name="Box_inertial_matrix" params="m l w h">
+       <inertial>
+               <mass value="${m}" />
+               <inertia ixx="${m*(h*h + l*l)/12}" ixy = "0" ixz = "0"
+                   iyy="${m*(w*w + l*l)/12}" iyz= "0"
+                   izz="${m*(w*w + h*h)/12}" />
+       </inertial>
+    </xacro:macro>
 	<link name="base_link">
 		<collision>
 			<origin xyz="0 0 0" rpy="0 0 0"/>
 			<geometry>
-				<box size="1.0 1.0 1.0"/>
+				<box size="${cam_size} ${cam_size} ${cam_size}"/>
 			</geometry>
 		</collision>
@@ -12,11 +21,8 @@
 			<origin xyz="0 0 0" rpy="0 0 0" />
 			<geometry>
-				<box size="1.0 1.0 1.0" />
+				<box size="${cam_size} ${cam_size} ${cam_size}" />
 			</geometry>
 		</visual>
-		<inertial>
-			<mass value="1.0" />
-			<inertia ixx="0.0833333" ixy = "0" ixz = "0" iyy="0.0833333" iyz= "0" izz="0.0833333" />
-		</inertial>
+        <xacro:Box_inertial_matrix m="1.0" l="${cam_size}" w="${cam_size}" h="${cam_size}"/>
 	</link>
 	<gazebo>
@@ -35,11 +41,11 @@
 		</plugin>
 	</gazebo>
-    <link name="imu_link"/>
+    <!-- <link name="imu_link"/>
     <joint name="imu_joint" type="fixed">
         <origin xyz="0.0 0.0 0.0" rpy="0 0 0"/>
         <parent link="base_link"/>
         <child link="imu_link"/>
-    </joint>
-    <gazebo>
+    </joint> -->
+    <!-- <gazebo>
         <plugin name="imu_controller" filename="libhector_gazebo_ros_imu.so">
             <updateRate>100.0</updateRate>
@@ -53,18 +59,14 @@
             <headingGaussianNoise>0.0</headingGaussianNoise>
         </plugin>
-    </gazebo>
-    <!-- velodyne and its parameters-->
-    <xacro:include filename="$(find obj_with_6dof)/urdf/velodyne.xacro"/>
-	<xacro:VLP name="rslidar16" topic="lidar_points" organize_cloud="true" hz="10" gpu="true" visualize="false">
-		<origin xyz="0.1 0.2 0.3" rpy="0 0 ${M_PI}" />
-	</xacro:VLP>
-    <!-- <xacro:include filename="$(find obj_with_6dof)/urdf/velodyne.xacro"/>
-	<xacro:VLP name="rslidar16" topic="lidar_points" organize_cloud="true" hz="10" gpu="true" visualize="false">
+    </gazebo> -->
+    <!-- avia and its parameters-->
+    <xacro:include filename="$(find obj6dof)/urdf/avia.xacro"/>
+	<xacro:Livox_AVIA name="avia" parent="base_link" visualize="false">
+		<origin xyz="0.05 0 0.1" rpy="0 0 0"/>
+	</xacro:Livox_AVIA>
+    <!-- camera and its parameters-->
+	<xacro:include filename="$(find obj6dof)/urdf/CameraSensor.xacro"/>
+	<xacro:Macro_CameraROS name="realsense" parent="base_link" frame="camera_fake" image_topic="image" fov="1.047198" hz="20" width="640" height="480">
 		<origin xyz="0 0 0" rpy="0 0 0" />
-	</xacro:VLP> -->
-    <!-- camera and its parameters-->
-	<!-- <xacro:include filename="$(find obj_with_6dof)/urdf/CameraSensor.xacro"/>
-	<xacro:Macro_CameraROS name="realsense" parent="base_link" frame="camera_fake" image_topic="image" fov="1.047198" hz="20" width="640" height="480">
-		<origin xyz="0.1 0.1 0.1" rpy="0 0 0" />
-	</xacro:Macro_CameraROS> -->
+	</xacro:Macro_CameraROS>
 </robot>
