Commit message: ✨ feat: avia done

File: urdf/avia.xacro (robot description, xacro)
@@ -17,9 +17,10 @@
         </inertial>
     </xacro:macro>
-    <xacro:macro name="Livox_Mid_gazebo_sensor" params="visualize:=True update_rate:=10 resolution:=0.002 noise_mean:=0.0 noise_stddev:=0.01 name:=avia">
+    <xacro:macro name="Livox_Mid_gazebo_sensor" params="visualize:=False update_rate:=10 resolution:=0.002 noise_mean:=0.0 noise_stddev:=0.01 name:=avia publish_pointcloud_type:=1">
         <gazebo reference="${name}">
             <sensor type="ray" name="laser_${name}">
                 <pose>0 0 0 0 0 0</pose>
-                <visualize>${visualize}</visualize>
+                <!-- Note: set gui to true and visualize True, so pointclouds are sent!! -->
+                <visualize>True</visualize>
                 <update_rate>${update_rate}</update_rate>
                 <!-- This ray plgin is only for visualization. -->
@@ -55,4 +56,5 @@
                     <downsample>${downsample}</downsample>
                     <csv_file_name>package://obj6dof/urdf/scan_mode/avia.csv</csv_file_name>
+                    <publish_pointcloud_type>${publish_pointcloud_type}</publish_pointcloud_type>
                     <ros_topic>${ros_topic}</ros_topic>
                 </plugin>
@@ -60,5 +62,5 @@
         </gazebo>
     </xacro:macro>
-    <xacro:macro name="Livox_AVIA" params="name:=livox parent:=base_link *origin visualize:=True">
+    <xacro:macro name="Livox_AVIA" params="name:=livox parent:=base_link *origin pctype">
         <link name="${name}">
             <xacro:null_inertial/>
@@ -81,5 +83,5 @@
             <xacro:insert_block name="origin"/>
         </joint>
-        <!-- <xacro:Livox_Mid_gazebo_sensor name="${name}" visualize="${visualize}"/> -->
+        <xacro:Livox_Mid_gazebo_sensor name="${name}" publish_pointcloud_type="${pctype}"/>
     </xacro:macro>
 </robot>

File: urdf/robot.urdf.xacro (robot description, xacro)
@@ -62,5 +62,5 @@
     <!-- avia and its parameters-->
     <xacro:include filename="$(find obj6dof)/urdf/avia.xacro"/>
-	<xacro:Livox_AVIA name="avia" parent="base_link" visualize="false">
+	<xacro:Livox_AVIA name="livox" parent="base_link" pctype="1">
 		<origin xyz="0.05 0 0.1" rpy="0 0 0"/>
 	</xacro:Livox_AVIA>

Commit message: ✨ feat:
mid360 done but pos need to be adjusted

File: urdf/avia.xacro (robot description, xacro)
@@ -19,5 +19,5 @@
     <xacro:macro name="Livox_Mid_gazebo_sensor" params="visualize:=False update_rate:=10 resolution:=0.002 noise_mean:=0.0 noise_stddev:=0.01 name:=avia publish_pointcloud_type:=1">
         <gazebo reference="${name}">
-            <sensor type="ray" name="laser_${name}">
+            <sensor type="ray" name="${name}">
                 <pose>0 0 0 0 0 0</pose>
                 <!-- Note: set gui to true and visualize True, so pointclouds are sent!! -->

File: urdf/robot.urdf.xacro (robot description, xacro)
@@ -61,11 +61,16 @@
     </gazebo> -->
     <!-- avia and its parameters-->
-    <xacro:include filename="$(find obj6dof)/urdf/avia.xacro"/>
-	<xacro:Livox_AVIA name="livox" parent="base_link" pctype="1">
-		<origin xyz="0.05 0 0.1" rpy="0 0 0"/>
-	</xacro:Livox_AVIA>
+    <!-- <xacro:include filename="$(find obj6dof)/urdf/avia.xacro"/>
+	<xacro:Livox_AVIA name="avia" parent="base_link" pctype="1">
+		<origin xyz="0.05 -0.09 0" rpy="0 0 0"/>
+	</xacro:Livox_AVIA> -->
+    <!-- mid360 and its parameters-->
+    <xacro:include filename="$(find obj6dof)/urdf/mid360.xacro"/>
+	<xacro:Livox_Mid360 name="mid360" parent="base_link" pctype="1">
+		<origin xyz="0.05 -0.09 0" rpy="0 0 0"/>
+	</xacro:Livox_Mid360>
     <!-- camera and its parameters-->
 	<xacro:include filename="$(find obj6dof)/urdf/CameraSensor.xacro"/>
-	<xacro:Macro_CameraROS name="realsense" parent="base_link" frame="camera_fake" image_topic="image" fov="1.047198" hz="20" width="640" height="480">
+	<xacro:Macro_CameraROS name="realsense" parent="base_link" frame="camera_fake" image_topic="image" fov="1.047198" hz="10" width="640" height="480">
 		<origin xyz="0 0 0" rpy="0 0 0" />
 	</xacro:Macro_CameraROS>

Commit message: ✨ feat:
test 2 avia done

File: urdf/avia.xacro (robot description, xacro)
@@ -6,7 +6,7 @@
     <xacro:property name="horizontal_fov" value="70.4"/>
     <xacro:property name="vertical_fov" value="77.2"/>
-    <xacro:property name="ros_topic" value="scan"/>
     <xacro:property name="samples" value="24000"/>
     <xacro:property name="downsample" value="1"/>
+    <xacro:property name="update_rate" value="10"/>
     <xacro:macro name="null_inertial">
         <inertial>
@@ -17,5 +17,5 @@
         </inertial>
     </xacro:macro>
-    <xacro:macro name="Livox_Mid_gazebo_sensor" params="visualize:=False update_rate:=10 resolution:=0.002 noise_mean:=0.0 noise_stddev:=0.01 name:=avia publish_pointcloud_type:=1">
+    <xacro:macro name="Livox_Mid_gazebo_sensor" params="visualize:=False name publish_pointcloud_type:=1 ros_topic">
         <gazebo reference="${name}">
             <sensor type="ray" name="${name}">
@@ -44,10 +44,10 @@
                             <min>${laser_min_range}</min>
                             <max>${laser_max_range}</max>
-                            <resolution>${resolution}</resolution>
+                            <resolution>0.01</resolution>
                         </range>
                         <noise>
                             <type>gaussian</type>
-                            <mean>${noise_mean}</mean>
-                            <stddev>${noise_stddev}</stddev>
+                            <mean>0.0</mean>
+                            <stddev>0.01</stddev>
                         </noise>
                     </ray>
@@ -62,5 +62,5 @@
         </gazebo>
     </xacro:macro>
-    <xacro:macro name="Livox_AVIA" params="name:=livox parent:=base_link *origin pctype">
+    <xacro:macro name="Livox_AVIA" params="name:=livox parent:=base_link *origin pctype ros_topic">
         <link name="${name}">
             <xacro:null_inertial/>
@@ -83,5 +83,5 @@
             <xacro:insert_block name="origin"/>
         </joint>
-        <xacro:Livox_Mid_gazebo_sensor name="${name}" publish_pointcloud_type="${pctype}"/>
+        <xacro:Livox_Mid_gazebo_sensor name="${name}" publish_pointcloud_type="${pctype}" ros_topic="${ros_topic}"/>
     </xacro:macro>
 </robot>

File: urdf/robot.urdf.xacro (robot description, xacro)
@@ -3,4 +3,7 @@
 	<xacro:property name="M_PI" value="3.14159265358979"/>
     <xacro:property name="cam_size" value="0.1"/>
+    <xacro:arg name="init_x" default="0"/>
+    <xacro:arg name="init_y" default="0"/>
+    <xacro:arg name="init_z" default="0.5"/>
     <xacro:macro name="Box_inertial_matrix" params="m l w h">
        <inertial>
@@ -29,4 +32,5 @@
 		<plugin name="move" filename="libSimMotion.so">
             <link>base_link</link>
+            <init_pos>$(arg init_x) $(arg init_y) $(arg init_z)</init_pos>
         </plugin>
 	</gazebo>
@@ -61,17 +65,10 @@
     </gazebo> -->
     <!-- avia and its parameters-->
-    <!-- <xacro:include filename="$(find obj6dof)/urdf/avia.xacro"/>
-	<xacro:Livox_AVIA name="avia" parent="base_link" pctype="1">
-		<origin xyz="0.05 -0.09 0" rpy="0 0 0"/>
-	</xacro:Livox_AVIA> -->
-    <!-- mid360 and its parameters-->
-    <xacro:include filename="$(find obj6dof)/urdf/mid360.xacro"/>
-	<xacro:Livox_Mid360 name="mid360" parent="base_link" pctype="1">
-		<origin xyz="0.05 -0.09 0" rpy="0 0 0"/>
-	</xacro:Livox_Mid360>
-    <!-- camera and its parameters-->
-	<xacro:include filename="$(find obj6dof)/urdf/CameraSensor.xacro"/>
-	<xacro:Macro_CameraROS name="realsense" parent="base_link" frame="camera_fake" image_topic="image" fov="1.047198" hz="10" width="640" height="480">
-		<origin xyz="0 0 0" rpy="0 0 0" />
-	</xacro:Macro_CameraROS>
+    <xacro:include filename="$(find obj6dof)/urdf/avia.xacro"/>
+	<xacro:Livox_AVIA name="avia1" parent="base_link" pctype="1" ros_topic="/avia1">
+		<origin xyz="0 0.1 0" rpy="0 0 ${M_PI/4}"/>
+	</xacro:Livox_AVIA>
+    <xacro:Livox_AVIA name="avia2" parent="base_link" pctype="1" ros_topic="/avia2">
+		<origin xyz="0 -0.1 0" rpy="0 0 -${M_PI/4}"/>
+	</xacro:Livox_AVIA>
 </robot>
