Commit message: ✨ feat: ai-dr

File: urdf/CameraSensor.xacro (robot description, xacro)
@@ -44,5 +44,5 @@
                     <updateRate>${hz}</updateRate>
                     <cameraName>${name}</cameraName>
-                    <imageTopicName>${image_topic}</imageTopicName>
+                    <imageTopicName>/${image_topic}</imageTopicName>
                     <cameraInfoTopicName>camera_info</cameraInfoTopicName>
                     <frameName>${frame}</frameName>

File: urdf/robot.urdf.xacro (robot description, xacro)
@@ -27,5 +27,5 @@
 	<gazebo>
 		<plugin name="p3d" filename="libSimP3D.so">
-			<updateRate>50.0</updateRate>
+			<updateRate>100.0</updateRate>
 			<bodyName>base_link</bodyName>
 			<topicName>odom</topicName>
@@ -56,11 +56,15 @@
     <!-- velodyne and its parameters-->
     <xacro:include filename="$(find obj_with_6dof)/urdf/velodyne.xacro"/>
-	<xacro:VLP name="rslidar16" topic="lidar_points" organize_cloud="false" hz="10" gpu="true" visualize="false">
-		<origin xyz="0.1 0.2 0.5" rpy="0 0 0" />
+	<xacro:VLP name="rslidar16" topic="lidar_points" organize_cloud="true" hz="10" gpu="true" visualize="false">
+		<origin xyz="0.1 0.2 0.3" rpy="0 0 ${M_PI}" />
 	</xacro:VLP>
+    <!-- <xacro:include filename="$(find obj_with_6dof)/urdf/velodyne.xacro"/>
+	<xacro:VLP name="rslidar16" topic="lidar_points" organize_cloud="true" hz="10" gpu="true" visualize="false">
+		<origin xyz="0 0 0" rpy="0 0 0" />
+	</xacro:VLP> -->
     <!-- camera and its parameters-->
-	<xacro:include filename="$(find obj_with_6dof)/urdf/CameraSensor.xacro"/>
+	<!-- <xacro:include filename="$(find obj_with_6dof)/urdf/CameraSensor.xacro"/>
 	<xacro:Macro_CameraROS name="realsense" parent="base_link" frame="camera_fake" image_topic="image" fov="1.047198" hz="20" width="640" height="480">
 		<origin xyz="0.1 0.1 0.1" rpy="0 0 0" />
-	</xacro:Macro_CameraROS>
+	</xacro:Macro_CameraROS> -->
 </robot>

Commit message: ✨ feat:
finish avia and mid360 launching at city, first version!

File: urdf/CameraSensor.xacro (robot description, xacro)
@@ -16,7 +16,7 @@
             <origin xyz="0 0 0" rpy="-${M_PI/2} 0 -${M_PI/2}"/>
             <parent link="${frame}"/>
-            <child link="camera"/>
+            <child link="${frame}/camera"/>
         </joint>
-        <link name="camera" />
+        <link name="${frame}/camera" />
         <gazebo reference="${frame}">
             <sensor type="camera" name="${name}">
@@ -31,5 +31,5 @@
                     </image>
                     <clip>
-                        <near>0.8</near>
+                        <near>0.2</near>
                         <far>300</far>
                     </clip>
@@ -37,5 +37,5 @@
                         <type>gaussian</type>
                         <mean>0.0</mean>
-                        <stddev>0.007</stddev>
+                        <stddev>0.0001</stddev>
                     </noise>
                 </camera>
@@ -44,5 +44,5 @@
                     <updateRate>${hz}</updateRate>
                     <cameraName>${name}</cameraName>
-                    <imageTopicName>/${image_topic}</imageTopicName>
+                    <imageTopicName>${image_topic}</imageTopicName>
                     <cameraInfoTopicName>camera_info</cameraInfoTopicName>
                     <frameName>${frame}</frameName>

Commit message: 🐞 fix:
fix mid360 hov and clone some camera plugin code for further modification

File: urdf/CameraSensor.xacro (robot description, xacro)
@@ -40,5 +40,6 @@
                     </noise>
                 </camera>
-                <plugin name="camera_controller" filename="libgazebo_ros_camera.so">
+                <!-- <plugin name="camera_controller" filename="libgazebo_ros_camera.so"> -->
+                <plugin name="camera_controller" filename="libgz_cam.so">
                     <alwaysOn>true</alwaysOn>
                     <updateRate>${hz}</updateRate>

File: urdf/cam_mid360.urdf.xacro (robot description, xacro)
@@ -55,7 +55,7 @@
 		<origin xyz="0 0.02 0" rpy="0 0 ${M_PI/4}"/>
 	</xacro:Macro_CameraROS>
-    <xacro:include filename="$(find obj6dof)/urdf/CameraSensor.xacro"/>
+    <!-- <xacro:include filename="$(find obj6dof)/urdf/CameraSensor.xacro"/>
 	<xacro:Macro_CameraROS name="right_cam" parent="base_link" frame="right_cam" image_topic="image" fov="1.047198" hz="10" width="640" height="480">
 		<origin xyz="0 -0.02 0" rpy="0 0 -${M_PI/4}"/>
-	</xacro:Macro_CameraROS>
+	</xacro:Macro_CameraROS> -->
 </robot>

File: urdf/mid360.xacro (robot description, xacro)
@@ -7,4 +7,6 @@
     <xacro:property name="samples" value="24000"/>
     <xacro:property name="downsample" value="1"/>
+    <xacro:property name="horizontal_fov" value="360"/>
+    <xacro:property name="vertical_fov" value="180.0"/>
     <xacro:macro name="null_inertial">
         <inertial>
@@ -28,12 +30,12 @@
                                 <samples>100</samples>
                                 <resolution>1</resolution>
-                                <min_angle>${-M_PI}</min_angle>
-                                <max_angle>${M_PI}</max_angle>
+                                <min_angle>${-horizontal_fov/360*M_PI}</min_angle>
+                                <max_angle>${horizontal_fov/360*M_PI}</max_angle>
                             </horizontal>
                             <vertical>
-                                <samples>360</samples>
+                                <samples>50</samples>
                                 <resolution>1</resolution>
-                                <min_angle>${-7.22/180*M_PI}</min_angle>
-                                <max_angle>${55.22/180*M_PI}</max_angle>
+                                <min_angle>${-vertical_fov/360*M_PI}</min_angle>
+                                <max_angle>${vertical_fov/360*M_PI}</max_angle>
                             </vertical>
                         </scan>

Commit message: 🐞 fix:
fix extrin and add intrin adapt to hik camera

File: urdf/CameraSensor.xacro (robot description, xacro)
@@ -2,22 +2,22 @@
 <robot xmlns:xacro="http://www.ros.org/wiki/xacro" name="Camera">
     <xacro:property name="camera_size" value="0.08"/>
-    <xacro:macro name="Macro_CameraROS" params="name parent frame image_topic hz *origin fov width height">
+    <xacro:macro name="Macro_CameraROS" params="name parent image_topic hz *origin fov width height">
         <joint name="${name}_mount_joint" type="fixed">
             <axis xyz="0 1 0"/>
             <xacro:insert_block name="origin"/>
             <parent link="${parent}"/>
-            <child link="${frame}"/>
+            <child link="${name}"/>
         </joint>
         <!-- gazebo camera frame -->
-        <link name="${frame}"/>
+        <link name="${name}"/>
         <!-- actual camera frame -->
         <joint name="${name}_mount_joint_1" type="fixed">
             <axis xyz="0 1 0"/>
             <origin xyz="0 0 0" rpy="-${M_PI/2} 0 -${M_PI/2}"/>
-            <parent link="${frame}"/>
-            <child link="${frame}/camera"/>
+            <parent link="${name}"/>
+            <child link="${name}/camera"/>
         </joint>
-        <link name="${frame}/camera" />
-        <gazebo reference="${frame}">
+        <link name="${name}/camera" />
+        <gazebo reference="${name}">
             <sensor type="camera" name="${name}">
                 <visualize>true</visualize>
@@ -47,11 +47,15 @@
                     <imageTopicName>${image_topic}</imageTopicName>
                     <cameraInfoTopicName>camera_info</cameraInfoTopicName>
-                    <frameName>${frame}</frameName>
-                    <hackBaseline>0.07</hackBaseline>
-                    <distortionK1>0.0</distortionK1>
-                    <distortionK2>0.0</distortionK2>
+                    <frameName>${name}</frameName>
+                    <hackBaseline>0.0</hackBaseline>
+                    <distortionK1>-0.0654429523802683</distortionK1>
+                    <distortionK2>0.0998393523310624</distortionK2>
                     <distortionK3>0.0</distortionK3>
-                    <distortionT1>0.0</distortionT1>
-                    <distortionT2>0.0</distortionT2>
+                    <distortionT1>0.00107153425553708</distortionT1>
+                    <distortionT2>-0.00283428566558518</distortionT2>
+                    <Cx>749.818357327634</Cx>
+                    <Cy>534.587402816582</Cy>
+                    <Fx>1311.05972093921</Fx>
+                    <Fy>1313.67270907052</Fy>
                 </plugin>
             </sensor>

File: urdf/cam_avia.urdf.xacro (robot description, xacro)
@@ -2,5 +2,5 @@
 <robot name="robot" xmlns:xacro="http://ros.org/wiki/xacro">
 	<xacro:property name="M_PI" value="3.14159265358979"/>
-    <xacro:property name="cam_size" value="0.1"/>
+    <xacro:property name="cam_size" value="0.01"/>
     <xacro:arg name="init_x" default="0"/>
     <xacro:arg name="init_y" default="0"/>
@@ -66,7 +66,13 @@
     <!-- avia and its parameters-->
     <xacro:include filename="$(find obj6dof)/urdf/avia.xacro"/>
+	<!-- <xacro:Livox_AVIA name="avia" parent="hik/camera" pctype="1"> -->
 	<xacro:Livox_AVIA name="avia" parent="base_link" pctype="1">
-		<origin xyz="0.05 -0.09 0" rpy="0 0 0"/>
+        <origin xyz="0 0 0.01" rpy="0 0 0"/>
 	</xacro:Livox_AVIA>
+    <!-- camera and its parameters-->
+	<xacro:include filename="$(find obj6dof)/urdf/CameraSensor.xacro"/>
+	<xacro:Macro_CameraROS name="hik" parent="avia" image_topic="image" fov="${M_PI*73.6/180}" hz="1" width="1536" height="1024">
+		<origin xyz="0.146255  0.288638  0.0275334" rpy="1.55921507 -0.02202108 -0.0168772" />
+	</xacro:Macro_CameraROS>
     <!-- mid360 and its parameters-->
     <!-- <xacro:include filename="$(find obj6dof)/urdf/mid360.xacro"/>
@@ -74,8 +80,3 @@
 		<origin xyz="0.05 -0.09 0" rpy="0 0 0"/>
 	</xacro:Livox_Mid360> -->
-    <!-- camera and its parameters-->
-	<xacro:include filename="$(find obj6dof)/urdf/CameraSensor.xacro"/>
-	<xacro:Macro_CameraROS name="realsense" parent="base_link" frame="camera_fake" image_topic="image" fov="1.047198" hz="10" width="640" height="480">
-		<origin xyz="0 0 0" rpy="0 0 0" />
-	</xacro:Macro_CameraROS>
 </robot>

Commit message: 🐞 fix: fix extrin

File: urdf/CameraSensor.xacro (robot description, xacro)
@@ -13,5 +13,5 @@
         <!-- actual camera frame -->
         <joint name="${name}_mount_joint_1" type="fixed">
-            <axis xyz="0 1 0"/>
+            <axis xyz="0 0 1"/>
             <origin xyz="0 0 0" rpy="-${M_PI/2} 0 -${M_PI/2}"/>
             <parent link="${name}"/>

File: urdf/cam_avia.urdf.xacro (robot description, xacro)
@@ -73,5 +73,6 @@
 	<xacro:include filename="$(find obj6dof)/urdf/CameraSensor.xacro"/>
 	<xacro:Macro_CameraROS name="hik" parent="avia" image_topic="image" fov="${M_PI*73.6/180}" hz="1" width="1536" height="1024">
-		<origin xyz="0.146255  0.288638  0.0275334" rpy="1.55921507 -0.02202108 -0.0168772" />
+		<origin xyz="-0.288638  -0.0275334  0.146255" rpy="-1.54897219  0.01713104 -0.01158016" />
+		<!-- <origin xyz="0 0 0" rpy="0 0 0" /> -->
 	</xacro:Macro_CameraROS>
     <!-- mid360 and its parameters-->
