Commit message: 🐳 chore: change a bit ext

File: urdf/cam_avia.urdf.xacro (robot description, xacro)
@@ -72,6 +72,7 @@
     <!-- camera and its parameters-->
 	<xacro:include filename="$(find obj6dof)/urdf/CameraSensor.xacro"/>
-	<xacro:Macro_CameraROS name="hik" parent="avia" image_topic="image" fov="${M_PI*73.6/180}" hz="1" width="1536" height="1024">
-		<origin xyz="-0.288638  -0.0275334  0.146255" rpy="-1.54897219  0.01713104 -0.01158016" />
+	<xacro:Macro_CameraROS name="hik" parent="avia" image_topic="image" fov="${M_PI*73.6/180}" hz="2" width="1536" height="1024">
+		<!-- <origin xyz="-0.288638  -0.0275334  0.146255" rpy="-1.54897219  0.01713104 -0.01158016" /> -->
+		<origin xyz="0 0.2 0" rpy="${-M_PI/2} 0 0" />
 		<!-- <origin xyz="0 0 0" rpy="0 0 0" /> -->
 	</xacro:Macro_CameraROS>
